File: hardware/trhmsx/trhmsx.kicad_pcb (KiCad board)
At the start: 4 copper layers, 150.4 x 120.4 mm, 127 parts, among them IC1 EPCS4, J1 MODULE-12V, J10 JOY2, J11 AudioJack2_Ground, J12 PJRAN1X1U02AUX, J13 CART2, J14 DH15, J15 JOY1, J16 CART1, J17 Conn_01x02, J2 ESP-01, J3 Barrel_Jack, J4 MICRO-SD, J5 Conn_01x02, J6 KEYBOARD-USB, J7 KEYBOARD-PS2, J8 Conn_02x05_Odd_Even, SW1 SW_DIP_x08, SW2 SW_Push, U1 EP1C12Q240C8N, U2 AMS1117-1.5, U3 AMS1117-3.3, U4 NC7WZU04P6X, U5 MT48LC16M16A2TG, U6 M51953BFP, Y1 21.47727 MHz

Commit message: v1.51 UPD2406
sync https://github.com/cristianoag/trhmsx
Parts:
- removed the G*** at (160.0, 181.2)
- removed J12: PJRAN1X1U02AUX, TRHMSX:SWITCHCRAFT_PJRAN1X1U02AUX
- removed the LOGO_MSX at (196.2, 135.2)
- removed R4, R6: 1K, Resistor_SMD:R_0805_2012Metric
- added C33: 3.3uF, Capacitor_SMD:C_0805_2012Metric, B.Cu at (240.7, 168.3)
- added C34: 3.3uF, Capacitor_SMD:C_0805_2012Metric, B.Cu at (240.7, 173.4)
- added C35: 10uF, Capacitor_SMD:C_0805_2012Metric, B.Cu at (244.3, 182.6)
- added D10: LED3, LED_SMD:LED_0805_2012Metric, F.Cu at (246.1, 174.2)
- added G***: LOGO, TRHMSX:LOGO_TRH, B.Cu at (160.3, 181.7)
- added J18: S-Video, TRHMSX:CUI_MD-40SM, F.Cu at (219.7, 74.8)
- added LOGO_MSX: , TRHMSX:LOGO_MSX, F.Cu at (196.7, 135.0)
- added R12: 1K, Resistor_SMD:R_0805_2012Metric, F.Cu at (241.0, 174.2)
- added R13: 2.2K, Resistor_SMD:R_0805_2012Metric, B.Cu at (264.4, 175.8)
- added R14: 2.2K, Resistor_SMD:R_0805_2012Metric, B.Cu at (258.7, 175.8)
- added SW3: SW_Push, Button_Switch_SMD:SW_Push_1P1T_NO_6x6mm_H9.5mm, F.Cu at (255.3, 171.7)
- added U7: CH559T, Package_SO:SSOP-20_5.3x7.2mm_P0.65mm, B.Cu at (247.7, 170.1)
- moved U6 2.28 mm to (259.8, 168.8), turned to 90 degrees
- moved C14 2.13 mm to (258.1, 163.1)
- moved C13 2.13 mm to (252.1, 163.1)
- moved REF** 1.87 mm to (176.7, 181.9)
- renumbered IC1 to U8
Connections:
- J6 pad 2: /KDAT -> Net-(J6-D-)
- J6 pad 3: /KCLK -> Net-(J6-D+)
Routing:
- net /VB_CV: track 54.5 -> 9.39 mm
- net +5V: track 382.3 -> 425.2 mm
- net /VG_SY: track 11.4 -> 41.1 mm
- net GND: track 151.5 -> 172.4 mm, vias 77 -> 81
- net /KDAT: track 117.3 -> 99.9 mm, vias 1 -> 3
- net Net-(U7-P4.6): track 0.00 -> 12.1 mm, vias 0 -> 1
- net /VR_SC: track 15.2 -> 26.8 mm
- net Net-(J6-D-): track 0.00 -> 11.1 mm
- net Net-(U6-DC): track 54.9 -> 44.2 mm, vias 1 -> 2
- net Net-(J6-D+): track 0.00 -> 10.4 mm
- net /RESET: track 187.9 -> 183.0 mm
- net /AS_CS: track 126.1 -> 130.5 mm
- net /KCLK: track 101.1 -> 105.4 mm, vias 1 -> 2
- net Net-(U1A-VCCA_PLL1): track 11.4 -> 15.6 mm
- net /MBA1: track 39.9 -> 43.9 mm
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Other:
- board text added: "${TITLE} - Rev ${REVISION}"
- board text removed: "Composite"
- board text removed: "Rev 1.3 - 03/2024"
