File: hardware/trhmsx/trhmsx.kicad_sch (KiCad schematic)
At the start: 124 parts, among them IC1 EPCS4, J1 MODULE-12V, J10 JOY2, J11 AudioJack2_Ground, J12 PJRAN1X1U02AUX, J13 CART2, J14 DH15, J15 JOY1, J16 CART1, J17 Conn_01x02, J2 ESP-01, J3 Barrel_Jack, J4 MICRO-SD, J5 Conn_01x02, J6 KEYBOARD-USB, J7 KEYBOARD-PS2, J8 Conn_02x05_Odd_Even, J9 EXPANSION, SW1 SW_DIP_x08, SW2 SW_Push, U1 EP1C12Q240C8N, U2 AMS1117-1.5, U3 AMS1117-3.3, U4 NC7WZU04P6X, U5 MT48LC16M16A2TG, U6 M51953BFP, Y1 21.47727 MHz

Commit message: v1.51 UPD2406
sync https://github.com/cristianoag/trhmsx
Parts:
- removed J12: PJRAN1X1U02AUX, TRHMSX:SWITCHCRAFT_PJRAN1X1U02AUX, symbol PJRAN1X1U02AUX:PJRAN1X1U02AUX
- removed R4, R6: 1K, Resistor_SMD:R_0805_2012Metric, symbol Device:R
- added C33, C34: 3.3uF, Capacitor_SMD:C_0805_2012Metric, symbol Device:C
- added C35: 10uF, Capacitor_SMD:C_0805_2012Metric, symbol Device:C
- added D10: LED3, LED_SMD:LED_0805_2012Metric, symbol Device:LED
- added J12: Composite, Connector_PinHeader_2.54mm:PinHeader_1x02_P2.54mm_Vertical, symbol Connector_Generic:Conn_01x02
- added J18: S-Video, TRHMSX:CUI_MD-40SM, symbol MD-40SM:MD-40SM
- added R12: 1K, Resistor_SMD:R_0805_2012Metric, symbol Device:R
- added R13, R14: 2.2K, Resistor_SMD:R_0805_2012Metric, symbol Device:R
- added SW3: SW_Push, Button_Switch_SMD:SW_Push_1P1T_NO_6x6mm_H9.5mm, symbol Switch:SW_Push
- added U7: CH559T, Package_SO:SSOP-20_5.3x7.2mm_P0.65mm, symbol CH55x:CH559T
- renumbered IC1 to U8
Connections:
- net +3.3V: now also C33.1, U7.20 (VDD33)
- net +5V: now also C34.1, C35.1, R12.1, R13.1, R14.1, U7.19 (VIN5)
- net GND: now also C33.2, C34.2, C35.2, J12.2 (Pin_2), J18.1, J18.2, J18.S1 (SHIELD), J18.S2 (SHIELD), J18.S3 (SHIELD), SW3.1, U7.10 (P4.7), U7.18 (GND)
- net KCLK: now also R14.2, U7.5 (P1.7/SCK); no longer J6.3 (D+)
- net KDAT: now also R13.2, U7.2 (P1.4/CS); no longer J6.2 (D-)
- net VB_CV: now also J12.1 (Pin_1)
- net VG_SY: now also J18.3
- net VR_SC: now also J18.4
- new net: SW3.2, U7.9 (P4.6)
- new net: D10.1 (K), U7.11 (PWM2/P2.5)
- new net: D10.2 (A), R12.2
- new net: J6.3 (D+), U7.14 (D+/P5.1)
- new net: J6.2 (D-), U7.15 (D-/P5.0)
- no-connect marks 35 -> 45
Other:
- moved on the sheet: C16, C17, C18, C19, C20, C21, C22, C23, D1, D2, D3, D4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
